Commit message: update robot description

File: robot_description/urdf/acemate.urdf (robot description, URDF)
Before this commit: robot acemate, 6 links, 5 joints
Links:
- added link base
Joints:
- added joint base_link-base_fixed_joint: type fixed, parent base_link, child base, origin xyz=0 0 0 rpy=0 0 0
